Commit message: Imported upstream version '1.0.9' of 'upstream'

File: summit_xl_description/robots/summit_xl.urdf.xacro (robot description, xacro)
@@ -48,12 +48,10 @@
   <!-- Hokuyo laser sensors can be parametized with min_angle and max_angle e.g: -->
   <!--xacro:sensor_hokuyo_utm30lx name="hokuyo_base" parent="base_link" min_angle="2.35" max_angle="-2.35"-->
-	<xacro:sensor_hokuyo_utm30lx name="hokuyo_base" parent="base_link">
+	<!--xacro:sensor_hokuyo_utm30lx name="hokuyo_base" parent="base_link">
 		<origin xyz="0.0 0.0 0.33" rpy="0 0 0"/>
-	</xacro:sensor_hokuyo_utm30lx>
-<!--
-	<xacro:sensor_hokuyo_urg04lx name="hokuyo1" parent="base_link">
-		<origin xyz="-0.1 0.0 0.33" rpy="0 0 0"/>
+	</xacro:sensor_hokuyo_utm30lx-->
+	<xacro:sensor_hokuyo_urg04lx name="hokuyo_base" parent="base_link">
+		<origin xyz="-0.0 0.0 0.33" rpy="0 0 0"/>
 	</xacro:sensor_hokuyo_urg04lx>
--->
 <!--
   <xacro:sensor_hokuyo_ust10lx name="hokuyo_base" parent="base_link">
@@ -61,7 +59,7 @@
 	</xacro:sensor_hokuyo_ust10lx>
 -->
-	<xacro:sensor_axis name="camera" parent="base_link">
+	<!--xacro:sensor_axis name="camera" parent="base_link">
 		<origin xyz="0.19 0 0.17" rpy="0 ${15*PI/180} 0"/>
-	</xacro:sensor_axis>
+	</xacro:sensor_axis-->
 	<xacro:sensor_imu name="imu" parent="base_link">
 		<origin xyz="-0.18 0.0 0.170" rpy="0 0 0"/>
@@ -70,9 +68,7 @@
 		<origin xyz="-0.22 0 0.275" rpy="0 0 0"/>
 	</xacro:sensor_gps>
-<!--
-	<xacro:sensor_asus_xtion_pro name="xtion_pro" parent="base_link">
-		<origin xyz="0.3 0.0 0.3" rpy="0 0 0"/>
-	</xacro:sensor_asus_xtion_pro>
--->
+	<xacro:sensor_orbbec_astra name="orbbec_astra" parent="base_link">
+		<origin xyz="0.324 0.012 0.172" rpy="0 0 0"/>
+	</xacro:sensor_orbbec_astra>
 <!--
 	<xacro:sensor_kinect name="kinect" parent="base_link">

Commit message: Imported upstream version '1.0.10' of 'upstream'

File: summit_xl_description/robots/summit_xl.urdf.xacro (robot description, xacro)
@@ -31,5 +31,5 @@
 	<!-- Gazebo skid steering pluggins -->
 	<!-- xacro:ros_force_based_move broadcastOdomTF="1"/ -->
-	<xacro:skid_steering broadcastOdomTF="1"/>
+	<xacro:skid_steering broadcastOdomTF="0"/>
 	<!-- WHEELS -->
 	<xacro:rubber_wheel name="front_right" parent="base_link" reflect="false" hq="${hq}">
@@ -62,7 +62,7 @@
 		<origin xyz="0.19 0 0.17" rpy="0 ${15*PI/180} 0"/>
 	</xacro:sensor_axis-->
-	<xacro:sensor_imu name="imu" parent="base_link">
+	<xacro:sensor_imu_hector name="imu" parent="base_link">
 		<origin xyz="-0.18 0.0 0.170" rpy="0 0 0"/>
-	</xacro:sensor_imu>
+	</xacro:sensor_imu_hector>
 	<xacro:sensor_gps name="gps" parent="base_link">
 		<origin xyz="-0.22 0 0.275" rpy="0 0 0"/>

File: summit_xl_description/urdf/bases/summit_xl_base.gazebo.xacro (robot description, xacro)
@@ -1,4 +1,4 @@
 <?xml version="1.0"?>
-<robot xmlns:xacro="http://ros.org/wiki/xacro">
+<robot xmlns:xacro="http://www.ros.org/wiki/xacro">
   <!-- ros control plugin -->
   <xacro:macro name="ros_control">

File: summit_xl_description/urdf/structures/structure_hokuyo.urdf.xacro (robot description, xacro)
@@ -4,5 +4,5 @@
 	  <joint name="${name}_joint" type="fixed">
 	    <axis xyz="0 1 0"/>
-	    <insert_block name="origin"/>
+	    <xacro:insert_block name="origin"/>
 	    <parent link="${parent}"/>
 	    <child link="${name}_link"/>

File: summit_xl_description/urdf/structures/structure_ptz_rgbd_gps.urdf.xacro (robot description, xacro)
@@ -4,5 +4,5 @@
 	  <joint name="${name}_joint" type="fixed">
 	    <axis xyz="0 1 0"/>
-	    <insert_block name="origin"/>
+	    <xacro:insert_block name="origin"/>
 	    <parent link="${parent}"/>
 	    <child link="${name}_link"/>

File: summit_xl_description/urdf/wheels/omni_wheel.urdf.xacro (robot description, xacro)
@@ -3,17 +3,17 @@
   <xacro:property name="M_PI" value="3.1415926535897931" />
   <!-- Wheels -->
-  <property name="wheel_radius" value="0.127" />
-  <property name="wheel_height" value="0.087" />
-  <property name="wheel_mass" value="6.5" /> <!-- in kg-->
-  <macro name="cylinder_inertia" params="m r h">
+  <xacro:property name="wheel_radius" value="0.127" />
+  <xacro:property name="wheel_height" value="0.087" />
+  <xacro:property name="wheel_mass" value="6.5" /> <!-- in kg-->
+  <xacro:macro name="cylinder_inertia" params="m r h">
     <inertia  ixx="${m*(3*r*r+h*h)/12}" ixy = "0" ixz = "0"
               iyy="${m*(3*r*r+h*h)/12}" iyz = "0"
               izz="${m*r*r/2}" />
-  </macro>
+  </xacro:macro>
   <xacro:macro name="omni_wheel" params="name parent *origin reflect hq">
     <joint name="joint_${name}_wheel" type="continuous">
       <parent link="${parent}"/>
       <child link="${name}_wheel"/>
-      <insert_block name="origin" />
+      <xacro:insert_block name="origin" />
       <axis xyz="0 1 0" rpy="0 0 0" />
       <limit effort="100" velocity="100"/>

File: summit_xl_description/urdf/wheels/rubber_wheel.urdf.xacro (robot description, xacro)
@@ -3,7 +3,7 @@
   <xacro:property name="M_PI" value="3.1415926535897931" />
   <!-- Wheels -->
-  <property name="wheel_radius" value="0.117" />
-  <property name="wheel_height" value="0.14" />
-  <property name="wheel_mass" value="6.5" /> <!-- in kg-->
+  <xacro:property name="wheel_radius" value="0.117" />
+  <xacro:property name="wheel_height" value="0.14" />
+  <xacro:property name="wheel_mass" value="6.5" /> <!-- in kg-->
   <xacro:macro name="cylinder_inertia" params="m r h">
     <inertia  ixx="${m*(3*r*r+h*h)/12}" ixy = "0" ixz = "0"
@@ -16,5 +16,5 @@
       <parent link="${parent}"/>
       <child link="${name}_wheel"/>
-      <insert_block name="origin" />
+      <xacro:insert_block name="origin" />
       <axis xyz="0 1 0" rpy="0 0 0" />
       <limit effort="100" velocity="100"/>
